File: 1.1.0/TestRadio/VirtualSense_RT.sch (KiCad schematic (older format))
At the start: 43 parts, among them P2 CONN_1, P3 CONN_1, P5 CONN_1, P6 CONN_1, P7 RS, P8 RS, Q1 MOS_N, Q2 MOS_N, Q4 MOS_N, U1 CC2520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

Commit message: created radio test layer
Parts:
- removed C11: 100n, symbol CSMALL
- removed P5, P6: CONN_1, symbol CONN_1
- removed P7, P8: RS, symbol CONN_1
- removed Q4: MOS_N, symbol MOS_N
- removed U4: DIPOLO_2_4_V1, symbol DIPOLO_2_4_V1
- added C10: 1p8, symbol CSMALL
- added C13: 1p, symbol CSMALL
- added C5: 82p, symbol CSMALL
- added C9: 1p5, symbol CSMALL
- added R5: R5, symbol CONN_1
- added R6: 0R, symbol R
- added U4: BALUN_ANTENNA_2GHZ4_TI, symbol BALUN_ANTENNA_2GHZ4_TI
- added U5: ANTENNA_EXT_2GHZ4, symbol ANTENNA_EXT_2GHZ4
- added U6: ANTENNA2GHZ4_TI, symbol ANTENNA2GHZ4_TI
- C7: value 1.5p -> 39p
- C8: value 1.5p -> 1p8
Connections:
- net labels removed: CC_GND
- wire segments 184 -> 218
- no-connect marks 7 -> 5
Other:
- note removed: "Fiducial"
- note removed: "OpenHardware logo"
