File: 1.1.0/TestAudioDSP/VirtualSense_TADSP_3.sch (KiCad schematic (older format))
At the start: 1 part

Commit message: schematics of audio DSP test layer OK, added module on audio DSP test layer brd
Parts:
- added C31, C33, C34, C35, C36: 100n, symbol CSMALL
- added C32: 1u, symbol CSMALL
- added C37: 10n, symbol CSMALL
- added L3: BLM18AG601SN1D, symbol FILTER
- added R29, R30: 0, symbol RSML
- added R31, R32: 10K, symbol RSML
- gave numbers to parts that had none: 1
Connections:
- net labels added: 3V3, AGND, ANA_LDO_OUT, GNDPWR, VCC_1V3, VCC_1V8
- wire segments 0 -> 97
- no-connect marks 0 -> 2
