File: 1.1.0/AudioDSP/VirtualSense_ADSP.sch (KiCad schematic (older format))
At the start: 40 parts, among them M1 MIC, P2 CONN_1, P3 CONN_1, P5 CONN_1, P6 CONN_1, P7 DSP, P8 uC, Q1 MOS_N, U2 TLV320AIC3204, U4 DSX321G_12MHZ

Commit message: remove VirtualSenseDSP layer from repository
Parts:
- removed BT2: 1V5, symbol BATTERY
- removed Q1: MOS_N, symbol MOS_N
- added BT1: BH2466, symbol BH2466
- added C? (x2): 47pF, symbol CSMALL
- added C? (x2): 1u, symbol CP1SMALL
- added JP1: USB-3V3, symbol BREAKER
- added L3: BLM18AG601SN1D, symbol FILTER
- added R? (x2): 33, symbol RSML
- added R?: 2, symbol RSML
- added U?: TPS76933, symbol TPS76933
- added USB1: USB-PLUG, symbol CONN_4
- CONN1: value VBAT -> 3V3
- DJ2235: renamed from U?; value SWITCH_DJ2235 -> SW1
- renumbered L2 to L1, L1 to L2
Connections:
- net labels added: 3V3_USB, AGND, USB_N, USB_P, VUSB
- net labels removed: VBAT
- wire segments 140 -> 166
- no-connect marks 18 -> 19
Other:
- moved on the sheet: BT1, C11, C21, C23, C7, CONN1, CONN2, DJ2235, L1, L2, M1, R1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
