File: 1.1.0/AudioDSP/VirtualSense_ADSP_2.sch (KiCad schematic (older format))
At the start: 39 parts, among them P10 DSP-SDA, P11 DSP-SCL, U5 C5535, U6 SD, U7 MICRO_SD, X1 32.768KHz

Commit message: remove VirtualSenseDSP layer from repository
Parts:
- removed C29: 10u, symbol CP1SMALL
- removed C30: 100n, symbol CSMALL
- removed R23, R24, R26, R27, R28: 10K, symbol RSML
- removed R25: NO, symbol RSML
- removed U6: SD, symbol MICRO_SD
- removed U7: MICRO_SD, symbol MICRO_SD
Connections:
- wire segments 134 -> 98
