File: 1.1.0/AudioDSP/VirtualSense_ADSP_3.sch (KiCad schematic (older format))
At the start: 12 parts, among them U5 C5535

Commit message: remove VirtualSenseDSP layer from repository
Parts:
- removed L3: BLM18AG601SN1D, symbol FILTER
- added C?: 100n, symbol CSMALL
- added C?: 10u, symbol CP1SMALL
- added R? (x5): 10K, symbol RSML
- added R?: NO, symbol RSML
- added SD1, SD2: MICRO_SD, symbol MICRO_SD
Connections:
- net labels added: SD_CLK, SD_CMD, SD_DATA0, SD_DATA1, SD_DATA2, SD_DATA3
- wire segments 98 -> 131
